File: Rover_PDB/digital_control.kicad_sch (KiCad schematic)
At the start: 0 parts

Commit message: added the schematic to digital
hi
Parts:
- added C1: C, symbol Device:C
- added M1: Fan, symbol Motor:Fan
- added Q1, Q2: PMOS, symbol Simulation_SPICE:PMOS
- added U1: Teensy4.1, symbol teensy:Teensy4.1
- added U2: MCP9808_MSOP, Package_SO:MSOP-8_3x3mm_P0.65mm, symbol Sensor_Temperature:MCP9808_MSOP
Connections:
- new net: C1.2, Q1.1 (D), Q2.3 (S), U1.46 (3V3), U2.8 (V_{DD})
- new net: M1.2 (-), Q2.1 (D)
- new net: U1.40 (18_A4_SDA), U2.1 (SDA)
- new net: U1.41 (19_A5_SCL), U2.2 (SCL)
- new net +24V: M1.1 (+), Q1.3 (S)
- new net +5V: U1.48 (VIN)
- new net GND: C1.1, U1.47 (GND), U2.4 (GND)
