File: Rover_PDB/teensy/teensy.kicad_pcb (KiCad board)
At the start: 2 copper layers, 14 parts, among them J1 Conn_01x04, J2 Conn_01x04, J3 Conn_01x04, M1 Fan, M2 Fan, M3 Fan, Q1 Q_NMOS, Q2 Q_NMOS, U1 Teensy4.1, U2 MCP9808_MSOP

Commit message: update
Parts:
- added C2: 100nF, Capacitor_SMD:C_01005_0402Metric, F.Cu at (94.8, 65.5)
- added C3: 50nF, Capacitor_SMD:C_01005_0402Metric, F.Cu at (108.3, 70.5)
- C1: footprint Package_TO_SOT_SMD:SOT-23-6 -> Capacitor_SMD:C_01005_0402Metric
- Q1, Q2: value Q_NMOS -> NMOS; footprint Package_TO_SOT_THT:TO-92_Inline -> Package_TO_SOT_THT:TO-220-3_Vertical
- R1, R2, R3: footprint Package_DIP:DIP-8_W7.62mm -> Resistor_SMD:R_01005_0402Metric
- moved J2 54.0 mm to (83.0, 30.0)
- moved J3 53.1 mm to (49.4, 81.9), turned to 90 degrees
- moved Q2 48.0 mm to (115.2, 80.0)
- moved J1 40.6 mm to (94.0, 110.0), turned to 180 degrees
- moved Q1 35.5 mm to (103.0, 80.0)
- moved M3 32.4 mm to (125.5, 52.0)
- moved R1 30.5 mm to (97.0, 73.0)
- moved U1 30.1 mm to (70.6, 68.3), turned to 90 degrees
- moved M2 24.9 mm to (113.5, 52.0)
- moved R2 24.7 mm to (102.3, 63.5)
- moved M1 24.3 mm to (101.8, 52.0)
- moved U2 18.4 mm to (90.5, 68.1), turned to 90 degrees
- moved C1 12.2 mm to (84.9, 77.0)
- moved R3 12.0 mm to (89.2, 79.0)
Connections:
- Q1 pad 1: (no net) -> Net-(Q1-D)
- Q1 pad 2: (no net) -> Net-(Q1-G)
- Q1 pad 3: (no net) -> GND
- Q2 pad 1: (no net) -> Net-(M1--)
- Q2 pad 2: (no net) -> Net-(Q1-D)
- Q2 pad 3: (no net) -> GND
- R1 pad 2: Net-(Q1-PadG) -> Net-(Q1-G)
- R2 pad 2: Net-(Q1-PadD) -> Net-(Q1-D)
Routing:
- net Net-(U1-22_A8_CTX1): track 0.00 -> 60.9 mm, vias 0 -> 3
- net GND: track 0.00 -> 52.9 mm, vias 0 -> 6
- net Net-(U1-23_A9_CRX1_MCLK1): track 0.00 -> 48.2 mm, vias 0 -> 2
- net SCL_BMS_TEAM: track 0.00 -> 37.6 mm
- net Net-(M1-+): track 0.00 -> 35.3 mm
- net SDA_BMS_TEAM: track 0.00 -> 34.2 mm
- net Net-(J2-Pin_4): track 0.00 -> 31.9 mm, vias 0 -> 2
- net Net-(J2-Pin_3): track 0.00 -> 30.9 mm
- net Net-(J3-Pin_4): track 0.00 -> 30.2 mm
- net Net-(J3-Pin_3): track 0.00 -> 29.8 mm
- net Net-(M1--): track 0.00 -> 25.9 mm
- net Net-(J1-Pin_3): track 0.00 -> 25.5 mm, vias 0 -> 1
- net Net-(J1-Pin_4): track 0.00 -> 21.5 mm
- net Net-(U2-A0): track 0.00 -> 14.4 mm, vias 0 -> 2
- net Net-(Q1-D): track 0.00 -> 11.3 mm
