File: Rover_PDB/digital_control_work/teensy.kicad_sch (KiCad schematic)
At the start: 17 parts, among them J1 Conn_01x04, J2 Conn_01x04, J3 Conn_01x04, M1 Fan, M2 Fan, M3 Fan, Q1 NMOS, Q2 NMOS, U1 Teensy4.1, U2 MCP9808_MSOP

Commit message: circuit cleaning
pls pr properly im begging
Connections:
- net +3V3: now also J3.1 (Pin_1); no longer J1.4 (Pin_4), J2.4 (Pin_4), J3.4 (Pin_4)
- net GND: now also J3.2 (Pin_2); no longer C4.1, C4.2, J1.1 (Pin_1), J2.1 (Pin_1), J3.1 (Pin_1), U1.1 (GND), U1.48 (VIN), U1.52 (GND), U1.64 (GND)
- net SCL: no longer U1.41 (19_A5_SCL)
- net SCL_BMS_TEAM: no longer U1.16 (24_A10_TX6_SCL2)
- net SDA: no longer U1.40 (18_A4_SDA)
- net SDA_BMS_TEAM: no longer U1.17 (25_A11_RX6_SDA2)
- net at U1.10 (8_TX2_IN1): now also J3.4 (Pin_4); no longer J3.2 (Pin_2)
- net at U1.2 (0_RX1_CRX2_CS1): now also J1.3 (Pin_3); no longer J2.3 (Pin_3)
- net at U1.20 (28_RX7): now also J2.3 (Pin_3); no longer J1.3 (Pin_3)
- net at U1.21 (29_TX7): now also J2.4 (Pin_4); no longer J1.2 (Pin_2)
- net at U1.3 (1_TX1_CTX2_MISO1): now also J1.4 (Pin_4); no longer J2.2 (Pin_2)
- new net: C4.1, C4.2, U1.48 (VIN)
- no-connect marks 48 -> 57
Other:
- note added: "1: Vdd 2: Gnd 3: Tx 4: Rx"
- note removed: "1: Gnd 2: Rx 3: Tx 4: Vdd"
- moved on the sheet: J1, J2, J3

Commit message: thing
Parts:
- added J5, J6, J7: Conn_01x02, symbol Connector_Generic:Conn_01x02
- M1, M2, M3: footprint Connector_JST:JST_XH_B2B-XH-A_1x02_P2.50mm_Vertical -> TerminalBlock_RND:TerminalBlock_RND_205-00056_1x02_P5.00mm_45Degree
Connections:
- net GND: now also C4.1
- net SCL: now also U1.41 (19_A5_SCL), J5.1 (Pin_1)
- net SCL_BMS_TEAM: now also U1.38 (16_A2_RX4_SCL1), J6.1 (Pin_1)
- net SDA: now also U1.40 (18_A4_SDA), J5.2 (Pin_2)
- net SDA_BMS_TEAM: now also U1.39 (17_A3_TX4_SDA1), J6.2 (Pin_2)
- net SCL_POWER_MNG: now reaches U1.16 (24_A10_TX6_SCL2)
- net SCL_POWER_MNG: now also J7.1 (Pin_1)
- net SDA_POWER_MNG: now reaches U1.17 (25_A11_RX6_SDA2)
- net SDA_POWER_MNG: now also J7.2 (Pin_2)
- net at C4.2, U1.48 (VIN): no longer C4.1
- no-connect marks 57 -> 51
Other:
- note added: "Science"
