File: pdb/Rover_PDB.kicad_pcb (KiCad board)
At the start: 2 copper layers, 130.4 x 130.6 mm, 27 parts, among them J1 Conn_01x04, J2 Conn_01x04, J3 Conn_01x04, J4 Conn_01x04, J6 Conn_01x02, J7 Conn_01x02, M1 Fan, M2 Fan, M3 Fan, Q1 NMOS, Q2 NMOS, U1 Teensy4.1, U2 MCP9808_MSOP

Commit message: changes to pcb
Parts:
- moved UART_1 68.6 mm to (131.0, 161.0)
- moved UART_2 66.2 mm to (150.5, 120.5)
- moved SPI_1 66.1 mm to (151.5, 97.0)
- moved UART_3 62.9 mm to (151.5, 59.0)
- moved I2C_2 62.6 mm to (149.0, 76.5)
- renumbered J6 to I2C_1, J7 to I2C_2, J4 to SPI_1, J1 to UART_1, J3 to UART_2, J2 to UART_3
Routing:
- net +3V3: track 104.6 -> 325.3 mm
- net Net-(U1-1_TX1_CTX2_MISO1): track 20.5 -> 127.3 mm
- net Net-(U1-0_RX1_CRX2_CS1): track 22.5 -> 128.4 mm
- net Net-(U1-7_RX2_OUT1A): track 7.61 -> 82.0 mm
- net Net-(U1-28_RX7): track 0.00 -> 74.3 mm
- net Net-(U1-29_TX7): track 0.00 -> 71.8 mm
- net MOSI0: track 6.84 -> 78.4 mm
- net MISO0: track 6.17 -> 77.5 mm
- net CS0: track 7.23 -> 77.9 mm
- net SCK0: track 23.5 -> 94.2 mm
- net Net-(U1-8_TX2_IN1): track 14.7 -> 81.8 mm, vias 0 -> 1
- net SCL_2: track 6.13 -> 72.0 mm
- net SDA_2: track 5.93 -> 71.6 mm, vias 0 -> 1
- net GND: track 11.1 -> 41.1 mm, vias 8 -> 11

Commit message: added  resistor value and etc
Parts:
- R6: value R_Small_US -> 10k
Connections:
- R6 pad 1: Net-(C2-Pad1) -> Net-(U1-22_A8_CTX1)
- R6 pad 2: Net-(U1-22_A8_CTX1) -> GND
Changed lines of the file:
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@@
 			)
 		)
-		(property "Value" "R_Small_US"
+		(property "Value" "10k"
 			(at 0 1 0)
 			(layer "F.Fab")
@@
 			(layers "F.Cu" "F.Mask")
 			(roundrect_rratio 0.25)
-			(net "Net-(C2-Pad1)")
+			(net "Net-(U1-22_A8_CTX1)")
 			(pintype "passive")
 		)
@@
 			(layers "F.Cu" "F.Mask")
 			(roundrect_rratio 0.25)
-			(net "Net-(U1-22_A8_CTX1)")
+			(net "GND")
 			(pintype "passive")
 		)
