File: pdb/digital_control.kicad_sch (KiCad schematic)
At the start: 27 parts, among them J1 Conn_01x04, J2 Conn_01x04, J3 Conn_01x04, J4 Conn_01x04, J6 Conn_01x02, J7 Conn_01x02, M1 Fan, M2 Fan, M3 Fan, Q1 NMOS, Q2 NMOS, U1 Teensy4.1, U2 MCP9808_MSOP

Commit message: digital part of pcb
Parts:
- D1: footprint (none) -> Diode_SMD:D_01005_0402Metric
- J4: footprint (none) -> Connector:FanPinHeader_1x04_P2.54mm_Vertical
- J6, J7: footprint (none) -> Connector_JST:JST_PH_S2B-PH-K_1x02_P2.00mm_Horizontal
- R10, R4, R5, R7, R8, R9: footprint (none) -> Resistor_SMD:R_01005_0402Metric
- R6: footprint Package_DIP:DIP-8_W7.62mm -> Resistor_SMD:R_01005_0402Metric

Commit message: changes to pcb
Parts:
- renumbered J6 to I2C_1, J7 to I2C_2, J4 to SPI_1, J1 to UART_1, J3 to UART_2, J2 to UART_3
Changed lines of the file:
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@@
 		(dnp no)
 		(fields_autoplaced yes)
-		(property "Reference" "J2"
+		(property "Reference" "UART_3"
 			(at 44.45 119.3801 0)
-			(hide yes)
 			(show_name no)
 			(do_not_autoplace no)
@@
 			(project "Rover_PDB"
 				(path "/1d8f27e2-b230-4ef2-93e1-1a59415140e6/3b0a8c82-c99b-49b6-94bc-5fcff51bb6a4"
-					(reference "J2")
+					(reference "UART_3")
 					(unit 1)
 				)
@@
 		(dnp no)
 		(fields_autoplaced yes)
-		(property "Reference" "J7"
+		(property "Reference" "I2C_2"
 			(at 46.99 34.2899 0)
 			(show_name no)
@@
 			(project "Rover_PDB"
 				(path "/1d8f27e2-b230-4ef2-93e1-1a59415140e6/3b0a8c82-c99b-49b6-94bc-5fcff51bb6a4"
-					(reference "J7")
+					(reference "I2C_2")
 					(unit 1)
 				)
@@
 		(dnp no)
 		(fields_autoplaced yes)
-		(property "Reference" "J4"
+		(property "Reference" "SPI_1"
 			(at 86.36 26.6699 0)
 			(show_name no)
@@
 			(project "Rover_PDB"
 				(path "/1d8f27e2-b230-4ef2-93e1-1a59415140e6/3b0a8c82-c99b-49b6-94bc-5fcff51bb6a4"
-					(reference "J4")
+					(reference "SPI_1")
 					(unit 1)
 				)
@@
 		(in_pos_files yes)
 		(dnp no)
-		(property "Reference" "J3"
+		(property "Reference" "UART_2"
 			(at 31.75 90.17 90)
 			(show_name no)
@@
 			(project "Rover_PDB"
 				(path "/1d8f27e2-b230-4ef2-93e1-1a59415140e6/3b0a8c82-c99b-49b6-94bc-5fcff51bb6a4"
-					(reference "J3")
+					(reference "UART_2")
 					(unit 1)
 				)
@@
 		(in_pos_files yes)
 		(dnp no)
-		(property "Reference" "J1"
+		(property "Reference" "UART_1"
 			(at 40.894 72.136 90)
 			(show_name no)
@@
 			(project "Rover_PDB"
 				(path "/1d8f27e2-b230-4ef2-93e1-1a59415140e6/3b0a8c82-c99b-49b6-94bc-5fcff51bb6a4"
-					(reference "J1")
+					(reference "UART_1")
 					(unit 1)
 				)
@@
 		(dnp no)
 		(fields_autoplaced yes)
-		(property "Reference" "J6"
+		(property "Reference" "I2C_1"
 			(at 46.99 24.1299 0)
 			(show_name no)
@@
 			(project "Rover_PDB"
 				(path "/1d8f27e2-b230-4ef2-93e1-1a59415140e6/3b0a8c82-c99b-49b6-94bc-5fcff51bb6a4"
-					(reference "J6")
-					(unit 1)
-				)
+					(reference "I2C_1")
+					(unit 1)
+				)

Commit message: added  resistor value and etc
Parts:
- removed C2: 100nF, Capacitor_SMD:C_01005_0402Metric, symbol Device:C_Small
- R6: value R_Small_US -> 10k
Connections:
- net GND: now also R6.2
- net at R1.1, U1.44 (22_A8_CTX1): now also R6.1; no longer R6.2
Other:
- moved on the sheet: R6
Changed lines of the file:
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@@
 	)
 	(junction
-		(at 160.02 76.2)
-		(diameter 0)
-		(color 0 0 0 0)
-	)
-	(junction
 		(at 137.16 114.3)
 		(diameter 0)
@@
 	)
 	(junction
+		(at 165.1 76.2)
+		(diameter 0)
+		(color 0 0 0 0)
+	)
+	(junction
 		(at 135.89 101.6)
 		(diameter 0)
@@
 	(wire
 		(pts
-			(xy 119.38 76.2) (xy 160.02 76.2)
+			(xy 119.38 76.2) (xy 165.1 76.2)
 		)
 		(stroke
@@
 	(wire
 		(pts
-			(xy 160.02 76.2) (xy 165.1 76.2)
-		)
-		(stroke
-			(width 0)
-			(type default)
-		)
-	)
-	(wire
-		(pts
 			(xy 39.37 26.67) (xy 30.48 26.67)
 		)
@@
 	(wire
 		(pts
-			(xy 160.02 69.85) (xy 160.02 76.2)
-		)
-		(stroke
-			(width 0)
-			(type default)
-		)
-	)
-	(wire
-		(pts
 			(xy 62.23 99.06) (xy 63.5 99.06)
 		)
@@
 	(wire
 		(pts
-			(xy 160.02 60.96) (xy 160.02 64.77)
-		)
-		(stroke
-			(width 0)
-			(type default)
-		)
-	)
-	(wire
-		(pts
 			(xy 63.5 144.78) (xy 63.5 146.05)
 		)
@@
 	(wire
 		(pts
-			(xy 38.1 78.74) (xy 38.1 81.28)
+			(xy 175.26 76.2) (xy 179.07 76.2)
 		)
 		(stroke
@@
 	(wire
 		(pts
-			(xy 119.38 66.04) (xy 128.27 66.04)
+			(xy 38.1 78.74) (xy 38.1 81.28)
 		)
 		(stroke
@@
 	(wire
 		(pts
-			(xy 120.65 86.36) (xy 119.38 86.36)
+			(xy 119.38 66.04) (xy 128.27 66.04)
 		)
 		(stroke
@@
 	(wire
 		(pts
-			(xy 160.02 60.96) (xy 165.1 60.96)
+			(xy 120.65 86.36) (xy 119.38 86.36)
 		)
 		(stroke
@@
 	(wire
 		(pts
+			(xy 165.1 76.2) (xy 170.18 76.2)
+		)
+		(stroke
+			(width 0)
+			(type default)
+		)
+	)
+	(wire
+		(pts
 			(xy 52.07 114.3) (xy 63.5 114.3)
 		)
@@
 	(wire
 		(pts
-			(xy 165.1 66.04) (xy 165.1 67.31)
+			(xy 62.23 104.14) (xy 63.5 104.14)
 		)
 		(stroke
@@
 	(wire
 		(pts
-			(xy 62.23 104.14) (xy 63.5 104.14)
+			(xy 172.72 110.49) (xy 173.99 110.49)
 		)
 		(stroke
@@
 	(wire
 		(pts
-			(xy 172.72 110.49) (xy 173.99 110.49)
+			(xy 52.07 68.58) (xy 63.5 68.58)
 		)
 		(stroke
@@
 	(wire
 		(pts
-			(xy 52.07 68.58) (xy 63.5 68.58)
+			(xy 58.42 144.78) (xy 63.5 144.78)
 		)
 		(stroke
@@
 	(wire
 		(pts
-			(xy 58.42 144.78) (xy 63.5 144.78)
+			(xy 137.16 114.3) (xy 137.16 118.11)
 		)
 		(stroke
@@
 	(wire
 		(pts
-			(xy 137.16 114.3) (xy 137.16 118.11)
+			(xy 179.07 76.2) (xy 179.07 78.74)
 		)
 		(stroke
@@
 	(symbol
 		(lib_id "Device:R_Small_US")
-		(at 160.02 67.31 0)
+		(at 172.72 76.2 90)
 		(unit 1)
 		(body_style 1)
@@
 		(dnp no)
 		(property "Reference" "R6"
-			(at 154.178 70.612 90)
+			(at 171.958 79.248 90)
 			(show_name no)
 			(do_not_autoplace no)
@@
 					(size 1.27 1.27)
 				)
-				(justify left)
+				(justify right)
 			)
 		)
-		(property "Value" "R_Small_US"
-			(at 156.718 70.612 90)
+		(property "Value" "10k"
+			(at 171.958 81.788 90)
 			(show_name no)
 			(do_not_autoplace no)
@@
 					(size 1.27 1.27)
 				)
-				(justify left)
+				(justify right)
 			)
 		)
 		(property "Footprint" "Resistor_SMD:R_01005_0402Metric"
-			(at 160.02 67.31 0)
+			(at 172.72 76.2 0)
 			(hide yes)
 			(show_name no)
@@
 		)
 		(property "Datasheet" ""
-			(at 160.02 67.31 0)
+			(at 172.72 76.2 0)
 			(hide yes)
 			(show_name no)
@@
 		)
 		(property "Description" "Resistor, small US symbol"
-			(at 160.02 67.31 0)
+			(at 172.72 76.2 0)
 			(hide yes)
 			(show_name no)
@@
 	)
 	(symbol
-		(lib_id "Device:C_Small")
-		(at 165.1 63.5 0)
-		(unit 1)
-		(body_style 1)
-		(exclude_from_sim no)
-		(in_bom yes)
-		(on_board yes)
-		(in_pos_files yes)
-		(dnp no)
-		(property "Reference" "C2"
-			(at 170.942 61.214 90)
-			(show_name no)
-			(do_not_autoplace no)
-			(effects
-				(font
-					(size 1.27 1.27)
-				)
-				(justify right)
-			)
-		)
-		(property "Value" "100nF"
-			(at 168.402 61.214 90)
-			(show_name no)
-			(do_not_autoplace no)
-			(effects
-				(font
-					(size 1.27 1.27)
-				)
-				(justify right)
-			)
-		)
-		(property "Footprint" "Capacitor_SMD:C_01005_0402Metric"
-			(at 165.1 63.5 0)
-			(hide yes)
-			(show_name no)
-			(do_not_autoplace no)
-			(effects
-				(font
-					(size 1.27 1.27)
-				)
-			)
-		)
-		(property "Datasheet" ""
-			(at 165.1 63.5 0)
-			(hide yes)
-			(show_name no)
-			(do_not_autoplace no)
-			(effects
-				(font
-					(size 1.27 1.27)
-				)
-			)
-		)
-		(property "Description" "Unpolarized capacitor, small symbol"
-			(at 165.1 73.66 0)
-			(hide yes)
-			(show_name no)
-			(do_not_autoplace no)
-			(effects
-				(font
-					(size 1.27 1.27)
-				)
-			)
-		)
-		(pin "1"
-		)
-		(pin "2"
-		)
-		(instances
-			(project "Rover_PDB"
-				(path "/1d8f27e2-b230-4ef2-93e1-1a59415140e6/3b0a8c82-c99b-49b6-94bc-5fcff51bb6a4"
-					(reference "C2")
-					(unit 1)
-				)
-			)
-		)
-	)
-	(symbol
 		(lib_id "Motor:Fan")
 		(at 195.58 109.22 0)
@@
 	(symbol
 		(lib_id "power:GND")
-		(at 165.1 67.31 0)
+		(at 179.07 78.74 0)
 		(unit 1)
 		(body_style 1)
@@
 		(fields_autoplaced yes)
 		(property "Reference" "#PWR011"
-			(at 165.1 73.66 0)
+			(at 179.07 85.09 0)
 			(hide yes)
 			(show_name no)
@@
 		)
 		(property "Value" "GND"
-			(at 165.1 72.39 0)
+			(at 179.07 83.82 0)
 			(show_name no)
 			(do_not_autoplace no)
@@
 		)
 		(property "Footprint" ""
-			(at 165.1 67.31 0)
+			(at 179.07 78.74 0)
 			(hide yes)
 			(show_name no)
@@
 		)
 		(property "Datasheet" ""
-			(at 165.1 67.31 0)
+			(at 179.07 78.74 0)
 			(hide yes)
 			(show_name no)
@@
 		)
 		(property "Description" "Power symbol creates a global label with name \"GND\" , ground"
-			(at 165.1 67.31 0)
+			(at 179.07 78.74 0)
 			(hide yes)
 			(show_name no)
